File: KiCad/Cubotronix.sch (KiCad schematic (older format))
At the start: 33 parts, among them J1 Vin, J2 ADC, J3 GPIO12, J4 GPIO15, P2 Battery, P5 USB-Serial, P6 I2C/1-W, SW1 Boot, SW2 Reset, U1 AP2114H-3.3TRG1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

Commit message: Update of sch
Parts:
- removed MK1: Mounting_Hole, Mounting_Holes:MountingHole_2.2mm_M2_Pad_Via, symbol Mounting_Hole
Other:
- note added: "Pinout"
- moved on the sheet: J2, J3, J4
Changed lines of the file:
@@
 LIBS:ESP8266
 LIBS:flex
-LIBS:Cubotronix-cache
 EELAYER 25 0
 EELAYER END
@@
 Sheet 1 1
 Title "Cubotronix"
-Date "29/03/2018"
-Rev "0.1"
+Date "18/04/2018"
+Rev "0.2"
 Comp "Eduardo Contreras"
 Comment1 ""
@@
 	1    0    0    -1
 $EndComp
-Text Label 6180 3645 0    60   ~ 0
+Text Label 6160 1815 0    60   ~ 0
 A0
 $Comp
 L GND #PWR014
 U 1 1 57D2307B
-P 5975 3915
-F 0 "#PWR014" H 5975 3665 50  0001 C CNN
-F 1 "GND" H 5975 3765 50  0000 C CNN
-F 2 "" H 5975 3915 50  0000 C CNN
-F 3 "" H 5975 3915 50  0000 C CNN
-	1    5975 3915
+P 5955 2085
+F 0 "#PWR014" H 5955 1835 50  0001 C CNN
+F 1 "GND" H 5955 1935 50  0000 C CNN
+F 2 "" H 5955 2085 50  0000 C CNN
+F 3 "" H 5955 2085 50  0000 C CNN
+	1    5955 2085
 	1    0    0    -1
 $EndComp
@@
 L +3.3V #PWR025
 U 1 1 58514B84
-P 5975 3680
-F 0 "#PWR025" H 5975 3530 50  0001 C CNN
-F 1 "+3.3V" H 5975 3820 50  0000 C CNN
-F 2 "" H 5975 3680 50  0000 C CNN
-F 3 "" H 5975 3680 50  0000 C CNN
-	1    5975 3680
+P 5955 1850
+F 0 "#PWR025" H 5955 1700 50  0001 C CNN
+F 1 "+3.3V" H 5955 1990 50  0000 C CNN
+F 2 "" H 5955 1850 50  0000 C CNN
+F 3 "" H 5955 1850 50  0000 C CNN
+	1    5955 1850
 	1    0    0    -1
 $EndComp
@@
 	500  4600 11200 4600
 Wire Wire Line
-	5975 3745 6315 3745
+	5955 1915 6295 1915
 Wire Wire Line
 	710  1430 860  1430
@@
 SCL/GPIO5
 $Comp
-L Mounting_Hole MK1
-U 1 1 5AD80612
-P 5955 815
-F 0 "MK1" H 5955 1015 50  0000 C CNN
-F 1 "Mounting_Hole" H 5955 940 50  0000 C CNN
-F 2 "Mounting_Holes:MountingHole_2.2mm_M2_Pad_Via" H 5955 815 50  0001 C CNN
-F 3 "" H 5955 815 50  0001 C CNN
-	1    5955 815
-	1    0    0    -1
-$EndComp
-$Comp
 L Conn_01x03 J2
 U 1 1 5AD80ABF
-P 6515 3745
-F 0 "J2" H 6515 3945 50  0000 C CNN
-F 1 "ADC" V 6615 3740 50  0000 C CNN
-F 2 "Pin_Headers:Pin_Header_Straight_1x03_Pitch2.54mm" H 6515 3745 50  0001 C CNN
-F 3 "" H 6515 3745 50  0001 C CNN
-	1    6515 3745
-	1    0    0    -1
-$EndComp
-Wire Wire Line
-	5975 3845 6315 3845
-Wire Wire Line
-	6315 3645 6180 3645
-Wire Wire Line
-	5975 3915 5975 3845
-Wire Wire Line
-	5975 3745 5975 3680
+P 6495 1915
+F 0 "J2" H 6495 2115 50  0000 C CNN
+F 1 "ADC" V 6595 1910 50  0000 C CNN
+F 2 "Pin_Headers:Pin_Header_Straight_1x03_Pitch2.54mm" H 6495 1915 50  0001 C CNN
+F 3 "" H 6495 1915 50  0001 C CNN
+	1    6495 1915
+	1    0    0    -1
+$EndComp
+Wire Wire Line
+	5955 2015 6295 2015
+Wire Wire Line
+	6295 1815 6160 1815
+Wire Wire Line
+	5955 2085 5955 2015
+Wire Wire Line
+	5955 1915 5955 1850
 $Comp
 L Conn_01x03 J3
 U 1 1 5AD82440
-P 7420 3760
-F 0 "J3" H 7420 3960 50  0000 C CNN
-F 1 "GPIO12" V 7515 3760 50  0000 C CNN
-F 2 "Pin_Headers:Pin_Header_Straight_1x03_Pitch2.54mm" H 7420 3760 50  0001 C CNN
-F 3 "" H 7420 3760 50  0001 C CNN
-	1    7420 3760
+P 7925 1915
+F 0 "J3" H 7925 2115 50  0000 C CNN
+F 1 "GPIO12" V 8020 1915 50  0000 C CNN
+F 2 "Pin_Headers:Pin_Header_Straight_1x03_Pitch2.54mm" H 7925 1915 50  0001 C CNN
+F 3 "" H 7925 1915 50  0001 C CNN
+	1    7925 1915
 	1    0    0    -1
 $EndComp
@@
 L Conn_01x03 J4
 U 1 1 5AD82523
-P 8340 3735
-F 0 "J4" H 8340 3935 50  0000 C CNN
-F 1 "GPIO15" V 8435 3735 50  0000 C CNN
-F 2 "Pin_Headers:Pin_Header_Straight_1x03_Pitch2.54mm" H 8340 3735 50  0001 C CNN
-F 3 "" H 8340 3735 50  0001 C CNN
-	1    8340 3735
+P 9545 1905
+F 0 "J4" H 9545 2105 50  0000 C CNN
+F 1 "GPIO15" V 9640 1905 50  0000 C CNN
+F 2 "Pin_Headers:Pin_Header_Straight_1x03_Pitch2.54mm" H 9545 1905 50  0001 C CNN
+F 3 "" H 9545 1905 50  0001 C CNN
+	1    9545 1905
 	1    0    0    -1
 $EndComp
@@
 L +3.3V #PWR030
 U 1 1 5AD82C28
-P 6785 3690
-F 0 "#PWR030" H 6785 3540 50  0001 C CNN
-F 1 "+3.3V" H 6785 3830 50  0000 C CNN
-F 2 "" H 6785 3690 50  0000 C CNN
-F 3 "" H 6785 3690 50  0000 C CNN
-	1    6785 3690
-	1    0    0    -1
-$EndComp
-Wire Wire Line
-	6785 3860 7220 3860
-Wire Wire Line
-	6785 3760 7220 3760
+P 7290 1845
+F 0 "#PWR030" H 7290 1695 50  0001 C CNN
+F 1 "+3.3V" H 7290 1985 50  0000 C CNN
+F 2 "" H 7290 1845 50  0000 C CNN
+F 3 "" H 7290 1845 50  0000 C CNN
+	1    7290 1845
+	1    0    0    -1
+$EndComp
+Wire Wire Line
+	7290 2015 7725 2015
+Wire Wire Line
+	7290 1915 7725 1915
 $Comp
 L GND #PWR031
 U 1 1 5AD82C99
-P 6785 3930
-F 0 "#PWR031" H 6785 3680 50  0001 C CNN
-F 1 "GND" H 6785 3780 50  0000 C CNN
-F 2 "" H 6785 3930 50  0000 C CNN
-F 3 "" H 6785 3930 50  0000 C CNN
-	1    6785 3930
-	1    0    0    -1
-$EndComp
-Wire Wire Line
-	6785 3690 6785 3760
-Wire Wire Line
-	6785 3860 6785 3930
+P 7290 2085
+F 0 "#PWR031" H 7290 1835 50  0001 C CNN
+F 1 "GND" H 7290 1935 50  0000 C CNN
+F 2 "" H 7290 2085 50  0000 C CNN
+F 3 "" H 7290 2085 50  0000 C CNN
+	1    7290 2085
+	1    0    0    -1
+$EndComp
+Wire Wire Line
+	7290 1845 7290 1915
+Wire Wire Line
+	7290 2015 7290 2085
 $Comp
 L +3.3V #PWR032
@@
 	1    0    0    -1
 $EndComp
-Text Label 6890 3660 0    60   ~ 0
+Text Label 7395 1815 0    60   ~ 0
 GPIO12
 Wire Wire Line
-	6890 3660 7220 3660
-Text Label 7795 3635 0    60   ~ 0
+	7395 1815 7725 1815
+Text Label 9000 1805 0    60   ~ 0
 GPIO15
 Wire Wire Line
-	7795 3635 8140 3635
+	9000 1805 9345 1805
 $Comp
 L +3.3V #PWR033
 U 1 1 5AD86815
-P 7625 3675
-F 0 "#PWR033" H 7625 3525 50  0001 C CNN
-F 1 "+3.3V" H 7625 3815 50  0000 C CNN
-F 2 "" H 7625 3675 50  0000 C CNN
-F 3 "" H 7625 3675 50  0000 C CNN
-	1    7625 3675
-	1    0    0    -1
-$EndComp
-Wire Wire Line
-	7625 3675 7625 3735
-Wire Wire Line
-	7625 3735 8140 3735
+P 8830 1845
+F 0 "#PWR033" H 8830 1695 50  0001 C CNN
+F 1 "+3.3V" H 8830 1985 50  0000 C CNN
+F 2 "" H 8830 1845 50  0000 C CNN
+F 3 "" H 8830 1845 50  0000 C CNN
+	1    8830 1845
+	1    0    0    -1
+$EndComp
+Wire Wire Line
+	8830 1845 8830 1905
+Wire Wire Line
+	8830 1905 9345 1905
 $Comp
 L GND #PWR034
 U 1 1 5AD86CCD
-P 7785 3905
-F 0 "#PWR034" H 7785 3655 50  0001 C CNN
-F 1 "GND" H 7785 3755 50  0000 C CNN
-F 2 "" H 7785 3905 50  0000 C CNN
-F 3 "" H 7785 3905 50  0000 C CNN
-	1    7785 3905
-	1    0    0    -1
-$EndComp
-Wire Wire Line
-	7785 3905 7785 3835
-Wire Wire Line
-	7785 3835 8140 3835
+P 8990 2075
+F 0 "#PWR034" H 8990 1825 50  0001 C CNN
+F 1 "GND" H 8990 1925 50  0000 C CNN
+F 2 "" H 8990 2075 50  0000 C CNN
+F 3 "" H 8990 2075 50  0000 C CNN
+	1    8990 2075
+	1    0    0    -1
+$EndComp
+Wire Wire Line
+	8990 2075 8990 2005
+Wire Wire Line
+	8990 2005 9345 2005
 Connection ~ 1565 6100
 Text Label 7655 5885 3    60   ~ 0
 SCL/GPIO5
+Text Notes 5680 710  0    60   ~ 0
+Pinout
 $EndSCHEMATC

Commit message: change on/off pin
Connections:
- net VCC: now also C1.1, JP1.2, U1.3 (IN)
Changed lines of the file:
@@
 LIBS:ESP8266
 LIBS:flex
+LIBS:Cubotronix-cache
 EELAYER 25 0
 EELAYER END
@@
 	600  6100 1285 6100
 Wire Wire Line
-	1565 6100 1565 6215
+	1565 5920 1565 6215
 Wire Wire Line
 	860  5950 860  6100
@@
 Text Notes 5680 710  0    60   ~ 0
 Pinout
+Wire Wire Line
+	1205 6100 1205 5920
+Wire Wire Line
+	1205 5920 1565 5920
+Connection ~ 1205 6100
 $EndSCHEMATC
